File: MEGA-SHIELD/optos.kicad_sch (KiCad schematic)
At the start: 17 parts, among them J5 Screw_Terminal_01x07, U3 PC817, U4 PC817, U5 PC817, U6 PC817

Commit message: develop: version 1.1
Parts:
- D5, D6, D7, D8: footprint LED_SMD:LED_1206_3216Metric_Pad1.42x1.75mm_HandSolder -> LED_SMD:LED_0603_1608Metric_Pad1.05x0.95mm_HandSolder
- J5: value Screw_Terminal_01x07 -> ENTRADAS OPTOS; footprint TerminalBlock_Phoenix:TerminalBlock_Phoenix_MPT-0,5-7-2.54_1x07_P2.54mm_Horizontal -> Connector_Phoenix_MC:PhoenixContact_MCV_1,5_8-G-3.81_1x08_P3.81mm_Vertical; symbol Connector:Screw_Terminal_01x07 -> Connector:Screw_Terminal_01x08
- R10, R11, R12, R13, R6, R7, R8, R9: footprint Resistor_SMD:R_0805_2012Metric_Pad1.20x1.40mm_HandSolder -> Resistor_SMD:R_0603_1608Metric_Pad0.98x0.95mm_HandSolder
- U3: value PC817 -> OPTO3
- U4: value PC817 -> OPTO4
- U5: value PC817 -> OPTO2
- U6: value PC817 -> OPTO1
Connections:
- net +12V: now also J5.4 (Pin_4); no longer J5.5 (Pin_5)
- net COM: now also J5.3 (Pin_3); no longer J5.6 (Pin_6)
- net GND: now also J5.2 (Pin_2); no longer J5.7 (Pin_7)
- net SIG1: now also J5.8 (Pin_8); no longer J5.1 (Pin_1)
- net SIG2: now also J5.7 (Pin_7); no longer J5.2 (Pin_2)
- net SIG3: now also J5.6 (Pin_6); no longer J5.3 (Pin_3)
- net SIG4: now also J5.5 (Pin_5); no longer J5.4 (Pin_4)
- new net +5V: J5.1 (Pin_1)
Other:
- moved on the sheet: D5, D6, D7, D8, R10, R11, R12, R13, R6, R7, R8, R9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
