File: MEGA-SHIELD/ER-PROMEGA-SHIELD.kicad_pcb (KiCad board)
At the start: 2 copper layers, 172.2 x 88.7 mm, 82 parts, among them J1 1x3, J10 12V, J11 Screw_Terminal_01x03, J12 Conn_01x03_Female, J13 Screw_Terminal_01x03, J14 Conn_01x03_Female, J15 Screw_Terminal_01x03, J16 Screw_Terminal_01x03, J17 Conn_01x03_Female, J18 Conn_01x03_Female, J19 ENTRADAS OPTOS, J2 Screw_Terminal_01x10, J3 Screw_Terminal_01x10, J4 Screw_Terminal_01x07, J5 Screw_Terminal_01x10, J6 Screw_Terminal_01x06, J7 Screw_Terminal_01x06, J8 Screw_Terminal_01x10, J9 Screw_Terminal_01x04, K1 Rele3, K2 Rele1, K3 Rele4, K4 Rele2, U1 ULN2003, U2 OPTO1, U3 OPTO2, U4 OPTO3, U5 OPTO4

Commit message: feat: revision final v1.2
Parts:
- removed kibuzzard-653EA38E: G***, kibuzzard-653EA38E
- removed kibuzzard-65BC3466: G***, kibuzzard-65BC3466
- removed kibuzzard-65BC3498: G***, kibuzzard-65BC3498
- removed kibuzzard-65BC34CA: G***, kibuzzard-65BC34CA
- removed kibuzzard-65BC34FE: G***, kibuzzard-65BC34FE
- removed kibuzzard-65BC3573: G***, kibuzzard-65BC3573
- removed kibuzzard-65BC35D6: G***, kibuzzard-65BC35D6
- removed kibuzzard-65BC363F: G***, kibuzzard-65BC363F
- removed kibuzzard-65BC3690: G***, kibuzzard-65BC3690
- removed kibuzzard-65BC36E0: G***, kibuzzard-65BC36E0
- removed kibuzzard-65BC3745: G***, kibuzzard-65BC3745
- removed kibuzzard-65BC3814 (x4): G***, kibuzzard-65BC3814
- added REF**: MountingHole_3.2mm_M3, MountingHole:MountingHole_3.2mm_M3, F.Cu at (218.7, 142.7)
- added REF**: MountingHole_3.2mm_M3, MountingHole:MountingHole_3.2mm_M3, F.Cu at (96.8, 77.0)
- added REF**: Symbol_Danger_CopperTop_Big, Symbol:Symbol_Danger_CopperTop_Big, F.Cu at (133.6, 99.8)
- added kibuzzard-65BE8B15: G***, kibuzzard-65BE8B15, F.Cu at (115.8, 126.5)
- added kibuzzard-65BE8BA4: G***, kibuzzard-65BE8BA4, F.Cu at (78.3, 136.6)
- added kibuzzard-65BE8BAF: G***, kibuzzard-65BE8BAF, F.Cu at (105.8, 136.8)
- added kibuzzard-65BE8BBD: G***, kibuzzard-65BE8BBD, F.Cu at (144.3, 137.2)
- added kibuzzard-65BE8BD6: G***, kibuzzard-65BE8BD6, F.Cu at (172.6, 137.2)
- added kibuzzard-65BE8C01: G***, kibuzzard-65BE8C01, F.Cu at (218.4, 146.6)
- added kibuzzard-65BE8C38: G***, kibuzzard-65BE8C38, F.Cu at (90.6, 70.3)
- added kibuzzard-65BE8C47: G***, kibuzzard-65BE8C47, F.Cu at (153.8, 70.2)
- added kibuzzard-65BE8C4E: G***, kibuzzard-65BE8C4E, F.Cu at (126.0, 70.0)
- added kibuzzard-65BE8C57: G***, kibuzzard-65BE8C57, F.Cu at (186.9, 69.8)
- added kibuzzard-65BE8C7C: G***, kibuzzard-65BE8C7C, F.Cu at (230.9, 78.2)
- added kibuzzard-65BE8C8A: G***, kibuzzard-65BE8C8A, F.Cu at (230.6, 96.0)
- added kibuzzard-65BE8C97: G***, kibuzzard-65BE8C97, F.Cu at (230.4, 113.0)
- added kibuzzard-65BE8CA3: G***, kibuzzard-65BE8CA3, F.Cu at (230.4, 131.3)
- added kibuzzard-65BE8F36: G***, kibuzzard-65BE8F36, F.Cu at (223.5, 69.1)
- moved C1 3.73 mm to (95.8, 87.6)
- moved C3 3.16 mm to (97.0, 118.6)
- moved J10 1.37 mm to (85.3, 117.6)
- moved kibuzzard-65BC37BD 0.64 mm to (183.9, 111.0)
- moved kibuzzard-65BC37BD 0.53 mm to (191.5, 111.0)
- moved kibuzzard-65BC37BD 0.24 mm to (176.3, 111.0)
- moved kibuzzard-65BC37BD 0.22 mm to (169.4, 110.7)
Routing:
- net Net-(J1-Pin_2): track 51.4 -> 46.0 mm
- net +5V: track 329.6 -> 332.0 mm
- net +12V: track 279.7 -> 278.6 mm
Other:
- board size 172.2 x 88.7 mm -> 171.2 x 88.7 mm
